Commit message: chore: rename urdf files

File: vendors/automationware/apps/awtube-urdfviz/awtube362010v3.urdf (robot description, URDF)
Before this commit: robot awtube32010v2, 7 links, 6 joints
Links:
- link base_link: mass 18 -> 1.95; geometry collision mesh filename=package://awtube362010v3/meshes/base_link.STL; visual mesh filename=package://awtube362010v3/meshes/base_link.STL
- link link1: mass 17.11 -> 16.69; geometry collision mesh filename=package://awtube362010v3/meshes/link1.STL; visual mesh filename=package://awtube362010v3/meshes/link1.STL
- link link2: mass 37.96 -> 39.11; geometry collision mesh filename=package://awtube362010v3/meshes/link2.STL; visual mesh filename=package://awtube362010v3/meshes/link2.STL
- link link3: mass 11.27 -> 11.63; geometry collision mesh filename=package://awtube362010v3/meshes/link3.STL; visual mesh filename=package://awtube362010v3/meshes/link3.STL
- link link4: mass 9.75 -> 10.12; geometry collision mesh filename=package://awtube362010v3/meshes/link4.STL; visual mesh filename=package://awtube362010v3/meshes/link4.STL
- link link5: mass 5.22 -> 5.53; geometry collision mesh filename=package://awtube362010v3/meshes/link5.STL; visual mesh filename=package://awtube362010v3/meshes/link5.STL
- link link6: geometry collision mesh filename=package://awtube362010v3/meshes/link6.STL; visual mesh filename=package://awtube362010v3/meshes/link6.STL
Joints:
- joint joint5: axis 0 0 -1 -> 0 0 1
